File: PCB/gh80-3003.kicad_pcb (KiCad board)
At the start: 2 copper layers, 444.1 x 145.3 mm, 359 parts, among them J1 Conn_01x01, J12 Alectardy98, J13 Conn_01x01, J14 Conn_01x01, J15 Conn_01x01, J2 SWD, J3 Conn_01x04_MountingPin, J4 USB_C, J5 Conn_01x01, J55 Conn_01x01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

Commit message: finished production files
Parts:
- added L5: LED, Alectardy98:CHERRY_MX_LED, F.Cu at (158.3, -120.3)
- added L5: LED, Alectardy98:CHERRY_MX_LED, F.Cu at (132.6, -120.7)
- added L5: LED, Alectardy98:CHERRY_MX_LED, F.Cu at (107.0, -120.6)
Other:
- board text added: "3.3V"
- board text added: "BOOT"
- board text added: "Gnd"
- board text added: "Reset"
- board text added: "SWCLK"
- board text added: "SWD"
